File: kria-k26-devboard/PoE.sch (KiCad schematic (older format))
At the start: 15 parts, among them IC1 TPS2378DDA

Commit message: Progress in PCB placement
Parts:
- renumbered C26 to C157, C205 to C158, C30 to C159, C31 to C160, C206 to C161, C32 to C162, C33 to C163, C34 to C164, D1 to D11, D2 to D12, D4 to D13, IC1 to IC2, R13 to R97, R14 to R98
Changed lines of the file:
@@
 P 2250 3250
 AR Path="/63C44BC2/6253A5C7" Ref="D?"  Part="1"
-AR Path="/63C44BC2/62525BE1/6253A5C7" Ref="D1"  Part="1"
-F 0 "D1" H 2600 3657 50  0000 C CNN
+AR Path="/63C44BC2/62525BE1/6253A5C7" Ref="D11"  Part="1"
+F 0 "D11" H 2600 3657 50  0000 C CNN
 F 1 "MB10S" H 2600 3566 50  0000 C CNN
 F 2 "antmicro-footprints:MB10S" H 1700 3200 50  0001 C CNN
@@
 P 2250 4250
 AR Path="/63C44BC2/6253A5CF" Ref="D?"  Part="1"
-AR Path="/63C44BC2/62525BE1/6253A5CF" Ref="D2"  Part="1"
-F 0 "D2" H 2600 4657 50  0000 C CNN
+AR Path="/63C44BC2/62525BE1/6253A5CF" Ref="D12"  Part="1"
+F 0 "D12" H 2600 4657 50  0000 C CNN
 F 1 "MB10S" H 2600 4566 50  0000 C CNN
 F 2 "antmicro-footprints:MB10S" H 1700 4200 50  0001 C CNN
@@
 P 3500 4050
 AR Path="/63C44BC2/6253A5D7" Ref="D?"  Part="1"
-AR Path="/63C44BC2/62525BE1/6253A5D7" Ref="D4"  Part="1"
-F 0 "D4" H 3550 4200 60  0000 R CNN
+AR Path="/63C44BC2/62525BE1/6253A5D7" Ref="D13"  Part="1"
+F 0 "D13" H 3550 4200 60  0000 R CNN
 F 1 "SMAJ58A-13-F" H 3850 3900 60  0000 R CNN
 F 2 "antmicro-footprints:DO-214AC" H 3700 4250 60  0001 L CNN
@@
 P 4200 3650
 AR Path="/63C44BC2/6253A5F4" Ref="R?"  Part="1"
-AR Path="/63C44BC2/62525BE1/6253A5F4" Ref="R13"  Part="1"
-F 0 "R13" V 4155 3720 60  0000 L CNN
+AR Path="/63C44BC2/62525BE1/6253A5F4" Ref="R97"  Part="1"
+F 0 "R97" V 4155 3720 60  0000 L CNN
 F 1 "R_24k9_0402" H 4200 3500 60  0001 C CNN
 F 2 "antmicro-footprints:0402-res" H 4400 3850 60  0001 L CNN
@@
 P 4200 4350
 AR Path="/63C44BC2/6253A5FD" Ref="R?"  Part="1"
-AR Path="/63C44BC2/62525BE1/6253A5FD" Ref="R14"  Part="1"
-F 0 "R14" V 4155 4420 60  0000 L CNN
+AR Path="/63C44BC2/62525BE1/6253A5FD" Ref="R98"  Part="1"
+F 0 "R98" V 4155 4420 60  0000 L CNN
 F 1 "R_63R4_0402" H 4200 4200 60  0001 C CNN
 F 2 "antmicro-footprints:0402-res" H 4400 4550 60  0001 L CNN
@@
 P 5750 4800
 AR Path="/63C44BC2/6253A612" Ref="#PWR?"  Part="1"
-AR Path="/63C44BC2/62525BE1/6253A612" Ref="#PWR019"  Part="1"
-F 0 "#PWR019" H 5750 4550 50  0001 C CNN
+AR Path="/63C44BC2/62525BE1/6253A612" Ref="#PWR0342"  Part="1"
+F 0 "#PWR0342" H 5750 4550 50  0001 C CNN
 F 1 "GNDD" H 5754 4645 50  0000 C CNN
 F 2 "" H 5750 4800 50  0001 C CNN
@@
 P 4650 3800
 AR Path="/63C44BC2/6253A62C" Ref="IC?"  Part="1"
-AR Path="/63C44BC2/62525BE1/6253A62C" Ref="IC1"  Part="1"
-F 0 "IC1" H 5150 4065 50  0000 C CNN
+AR Path="/63C44BC2/62525BE1/6253A62C" Ref="IC2"  Part="1"
+F 0 "IC2" H 5150 4065 50  0000 C CNN
 F 1 "TPS2378DDA" H 5150 3974 50  0000 C CNN
 F 2 "antmicro-footprints:SOIC127P600X170-9N" H 5500 3900 50  0001 L CNN
@@
 P 3950 4050
 AR Path="/63C44BC2/6253A644" Ref="C?"  Part="1"
-AR Path="/63C44BC2/62525BE1/6253A644" Ref="C26"  Part="1"
-F 0 "C26" V 3800 4000 60  0000 L CNN
+AR Path="/63C44BC2/62525BE1/6253A644" Ref="C157"  Part="1"
+F 0 "C157" V 3800 4000 60  0000 L CNN
 F 1 "C_100n_0805_100V" H 3950 3900 60  0001 C CNN
 F 2 "antmicro-footprints:0805-cap" H 4150 4250 60  0001 L CNN
@@
 	6350 4200 6350 4700
 $Comp
-L antmicroCapacitorsmisc:C_47u_16V_1206 C32
+L antmicroCapacitorsmisc:C_47u_16V_1206 C162
 U 1 1 6254E76E
 P 9050 3900
-F 0 "C32" H 9165 3945 60  0000 L CNN
+F 0 "C162" H 9165 3945 60  0000 L CNN
 F 1 "C_47u_16V_1206" H 9050 3750 60  0001 C CNN
 F 2 "antmicro-footprints:1206-cap" H 9250 4100 60  0001 L CNN
@@
 $EndComp
 $Comp
-L antmicroCapacitorsmisc:C_47u_16V_1206 C33
+L antmicroCapacitorsmisc:C_47u_16V_1206 C163
 U 1 1 6254ED87
 P 9600 3900
-F 0 "C33" H 9715 3945 60  0000 L CNN
+F 0 "C163" H 9715 3945 60  0000 L CNN
 F 1 "C_47u_16V_1206" H 9600 3750 60  0001 C CNN
 F 2 "antmicro-footprints:1206-cap" H 9800 4100 60  0001 L CNN
@@
 $EndComp
 $Comp
-L antmicroCapacitorsmisc:C_100n_0402_16V C34
+L antmicroCapacitorsmisc:C_100n_0402_16V C164
 U 1 1 6255055B
 P 10200 3900
-F 0 "C34" H 10315 3945 60  0000 L CNN
+F 0 "C164" H 10315 3945 60  0000 L CNN
 F 1 "C_100n_0402_16V" H 10200 3750 60  0001 C CNN
 F 2 "antmicro-footprints:0402-cap" H 10400 4100 60  0001 L CNN
@@
 Connection ~ 10200 3450
 $Comp
-L power:GND #PWR020
+L power:GND #PWR0343
 U 1 1 62590E73
 P 10200 4750
-F 0 "#PWR020" H 10200 4500 50  0001 C CNN
+F 0 "#PWR0343" H 10200 4500 50  0001 C CNN
 F 1 "GND" H 10205 4577 50  0000 C CNN
 F 2 "" H 10200 4750 50  0001 C CNN
@@
 POE_VC4
 $Comp
-L antmicroCapacitorsmisc:C_22u_2220_100V C205
+L antmicroCapacitorsmisc:C_22u_2220_100V C158
 U 1 1 6A074DA7
 P 6350 4050
-F 0 "C205" V 6400 3750 60  0000 L CNN
+F 0 "C158" V 6400 3750 60  0000 L CNN
 F 1 "C_22u_2220_100V" H 6350 3900 60  0001 C CNN
 F 2 "antmicro-footprints:2220-cap" H 6550 4250 60  0001 L CNN
@@
 $EndComp
 $Comp
-L antmicroCapacitorsmisc:C_22u_2220_100V C30
+L antmicroCapacitorsmisc:C_22u_2220_100V C159
 U 1 1 6A0791F7
 P 6550 4050
-F 0 "C30" V 6600 3750 60  0000 L CNN
+F 0 "C159" V 6600 3750 60  0000 L CNN
 F 1 "C_22u_2220_100V" H 6550 3900 60  0001 C CNN
 F 2 "antmicro-footprints:2220-cap" H 6750 4250 60  0001 L CNN
@@
 $EndComp
 $Comp
-L antmicroCapacitorsmisc:C_22u_2220_100V C31
+L antmicroCapacitorsmisc:C_22u_2220_100V C160
 U 1 1 6A0794FE
 P 6750 4050
-F 0 "C31" V 6800 3750 60  0000 L CNN
+F 0 "C160" V 6800 3750 60  0000 L CNN
 F 1 "C_22u_2220_100V" H 6750 3900 60  0001 C CNN
 F 2 "antmicro-footprints:2220-cap" H 6950 4250 60  0001 L CNN
@@
 $EndComp
 $Comp
-L antmicroCapacitorsmisc:C_22u_2220_100V C206
+L antmicroCapacitorsmisc:C_22u_2220_100V C161
 U 1 1 6A079825
 P 6950 4050
-F 0 "C206" V 7000 3750 60  0000 L CNN
+F 0 "C161" V 7000 3750 60  0000 L CNN
 F 1 "C_22u_2220_100V" H 6950 3900 60  0001 C CNN
 F 2 "antmicro-footprints:2220-cap" H 7150 4250 60  0001 L CNN
