File: kria-k26-devboard/clock.sch (KiCad schematic (older format))
At the start: 0 parts

Commit message: Fixes on Reset pagae, progress through clock sheet
Parts:
- added C? (x2): C_100n_0402, antmicro-footprints:0402-cap, symbol antmicroCapacitors0402:C_100n_0402
- added U?: DSC557-0333FI1, antmicro-footprints:MICROCHIP_QFN14_3.2X2.5, symbol antmicroClockTimingRealTimeClocks:DSC557-0333FI1
Connections:
- net labels added: GND, PS_3V3
- wire segments 0 -> 22
Other:
- note added: "2x100MHz LVDS"
Changed lines of the file:
@@
 $Descr A4 11693 8268
 encoding utf-8
-Sheet 15 19
+Sheet 13 19
 Title ""
 Date ""
@@
 Comment4 ""
 $EndDescr
-Text HLabel 1950 1800 0    50   Input ~ 0
+Text HLabel 3250 1750 2    50   Input ~ 0
 GTR_REFCLK3_P
-Text HLabel 1950 1900 0    50   Input ~ 0
+Text HLabel 3250 1850 2    50   Input ~ 0
 GTR_REFCLK3_N
-Text HLabel 1950 2000 0    50   Input ~ 0
+Text HLabel 3250 1950 2    50   Input ~ 0
 GTR_REFCLK3_C2M_P
-Text HLabel 1950 2100 0    50   Input ~ 0
+Text HLabel 3250 2050 2    50   Input ~ 0
 GTR_REFCLK3_C2M_N
+$Comp
+L antmicroClockTimingRealTimeClocks:DSC557-0333FI1 U?
+U 1 1 6245C94F
+P 1700 1600
+F 0 "U?" H 2475 503 60  0000 C CNN
+F 1 "DSC557-0333FI1" H 2475 397 60  0000 C CNN
+F 2 "antmicro-footprints:MICROCHIP_QFN14_3.2X2.5" H 3100 740 60  0001 C CNN
+F 3 "https://www.mouser.pl/datasheet/2/268/DSC557_03_Two_Output_PCIe_Gen1_2_3_4_Clock_Generat-1917017.pdf" H 1850 1450 60  0001 C CNN
+F 4 "Microchip Technology" H 1750 1700 50  0001 C CNN "Manufacturer"
+F 5 "DSC557-0333FI1" H 1700 1600 50  0001 C CNN "MPN"
+	1    1700 1600
+	1    0    0    -1
+$EndComp
+Wire Wire Line
+	3100 1750 3250 1750
+Wire Wire Line
+	3250 1850 3100 1850
+Wire Wire Line
+	3100 1950 3250 1950
+Wire Wire Line
+	3250 2050 3100 2050
+Wire Wire Line
+	1850 1750 1800 1750
+$Comp
+L antmicroCapacitors0402:C_100n_0402 C?
+U 1 1 6245FC31
+P 1450 1250
+F 0 "C?" H 1565 1295 60  0000 L CNN
+F 1 "C_100n_0402" H 1450 1100 60  0001 C CNN
+F 2 "antmicro-footprints:0402-cap" H 1650 1450 60  0001 L CNN
+F 3 "" H 1450 1250 50  0001 C CNN
+F 4 "Murata" H 1650 1650 60  0001 L CNN "Manufacturer"
+F 5 "GRM155R61H104KE14D" H 1650 1550 60  0001 L CNN "MPN"
+F 6 "100n" H 1565 1197 50  0000 L CNN "Val"
+	1    1450 1250
+	1    0    0    -1
+$EndComp
+$Comp
+L power:GND #PWR?
+U 1 1 6246203F
+P 2000 1350
+F 0 "#PWR?" H 2000 1100 50  0001 C CNN
+F 1 "GND" H 2005 1177 50  0000 C CNN
+F 2 "" H 2000 1350 50  0001 C CNN
+F 3 "" H 2000 1350 50  0001 C CNN
+	1    2000 1350
+	1    0    0    -1
+$EndComp
+Wire Wire Line
+	2000 1350 2000 1050
+Wire Wire Line
+	2000 1050 2300 1050
+Wire Wire Line
+	2300 1050 2300 1100
+Connection ~ 2500 950
+Wire Wire Line
+	1800 950  1800 1750
+Wire Wire Line
+	1800 950  2500 950
+Wire Wire Line
+	2600 950  2600 1100
+Wire Wire Line
+	2500 950  2600 950
+Wire Wire Line
+	2500 950  2500 1100
+Wire Wire Line
+	1450 1100 1450 950
+Wire Wire Line
+	1450 950  1800 950
+Connection ~ 1800 950
+$Comp
+L power:GND #PWR?
+U 1 1 6246365B
+P 1450 1450
+F 0 "#PWR?" H 1450 1200 50  0001 C CNN
+F 1 "GND" H 1455 1277 50  0000 C CNN
+F 2 "" H 1450 1450 50  0001 C CNN
+F 3 "" H 1450 1450 50  0001 C CNN
+	1    1450 1450
+	1    0    0    -1
+$EndComp
+Wire Wire Line
+	1450 1450 1450 1400
+$Comp
+L antmicroCapacitors0402:C_100n_0402 C?
+U 1 1 62463CDF
+P 1050 1250
+F 0 "C?" H 1165 1295 60  0000 L CNN
+F 1 "C_100n_0402" H 1050 1100 60  0001 C CNN
+F 2 "antmicro-footprints:0402-cap" H 1250 1450 60  0001 L CNN
+F 3 "" H 1050 1250 50  0001 C CNN
+F 4 "Murata" H 1250 1650 60  0001 L CNN "Manufacturer"
+F 5 "GRM155R61H104KE14D" H 1250 1550 60  0001 L CNN "MPN"
+F 6 "100n" H 1165 1197 50  0000 L CNN "Val"
+	1    1050 1250
+	1    0    0    -1
+$EndComp
+Wire Wire Line
+	1050 1100 1050 950
+$Comp
+L power:GND #PWR?
+U 1 1 62463D3C
+P 1050 1450
+F 0 "#PWR?" H 1050 1200 50  0001 C CNN
+F 1 "GND" H 1055 1277 50  0000 C CNN
+F 2 "" H 1050 1450 50  0001 C CNN
+F 3 "" H 1050 1450 50  0001 C CNN
+	1    1050 1450
+	1    0    0    -1
+$EndComp
+Wire Wire Line
+	1050 1450 1050 1400
+Wire Wire Line
+	1050 950  1450 950
+Connection ~ 1450 950
+Text GLabel 1000 950  0    50   Input ~ 0
+PS_3V3
+$Comp
+L power:GND #PWR?
+U 1 1 62464C95
+P 1800 2100
+F 0 "#PWR?" H 1800 1850 50  0001 C CNN
+F 1 "GND" H 1805 1927 50  0000 C CNN
+F 2 "" H 1800 2100 50  0001 C CNN
+F 3 "" H 1800 2100 50  0001 C CNN
+	1    1800 2100
+	1    0    0    -1
+$EndComp
+Wire Wire Line
+	1800 2100 1800 2050
+Wire Wire Line
+	1800 2050 1850 2050
+Text Notes 550  750  0    100  ~ 20
+2x100MHz LVDS
+Wire Wire Line
+	1000 950  1050 950
+Connection ~ 1050 950
 $EndSCHEMATC

Commit message: Finished clock sheet
Parts:
- added C? (x4): C_100n_0402, antmicro-footprints:0402-cap, symbol antmicroCapacitors0402:C_100n_0402
- added R? (x5): R_100R_0402, antmicro-footprints:0402-res, symbol antmicroResistors0402:R_100R_0402
- added U?: XLL736027.000000X, antmicro-footprints:Oscillator_SMD_IDT_JU6-6_7.0x5.0mm_P2.54mm, symbol antmicroOscillators:XLL736027.000000X
- added U?: SN65LVDS1DR, antmicro-footprints:SOIC-8_W3.9mm, symbol antmicroInterfaceDriversReceiversTransceivers:SN65LVDS1DR
- added Y?: AX3DAF1-125.0000, antmicro-footprints:AX3DAF1, symbol antmicroOscillators:AX3DAF1-125.0000
- added Y?: ECS-2520MVLC-260-CM-TR, antmicro-footprints:Oscillator_SMD_ECS_2520MV-xxx-xx-4Pin_2.5x2.0mm, symbol antmicroCrystals:ECS-2520MVLC-260-CM-TR
Connections:
- net labels added: GTR_REFCLK0_C2M_N, GTR_REFCLK0_C2M_P, GTR_REFCLK1_C2M_N, GTR_REFCLK1_C2M_P, GTR_REFCLK2_C2M_N, GTR_REFCLK2_C2M_P, PS_CLK_EN
- wire segments 22 -> 90
Other:
- note added: "DisplayPort GTH REFCLK: 27MHz LVDS"
- note added: "ETH GTH REFCLK: 125MHz LVDS"
- note added: "PCIe GTH REFCLK: 2x100MHz LVDS"
- note added: "USB GTH REFCLK: 26MHz LVDS"
- note removed: "2x100MHz LVDS"
- moved on the sheet: C?

Commit message: Added Led voltage indicator, fan circuit. Tidied up supply and SOM sheet
Parts:
- gave numbers to parts that had none: 16
Changed lines of the file:
@@
 GTR_REFCLK3_C2M_N
 $Comp
-L antmicroClockTimingRealTimeClocks:DSC557-0333FI1 U?
+L antmicroClockTimingRealTimeClocks:DSC557-0333FI1 U2
 U 1 1 6245C94F
 P 1950 1850
-F 0 "U?" H 2725 753 60  0000 C CNN
+F 0 "U2" H 2725 753 60  0000 C CNN
 F 1 "DSC557-0333FI1" H 2725 647 60  0000 C CNN
 F 2 "antmicro-footprints:MICROCHIP_QFN14_3.2X2.5" H 3350 990 60  0001 C CNN
@@
 	2100 2000 2050 2000
 $Comp
-L antmicroCapacitors0402:C_100n_0402 C?
+L antmicroCapacitors0402:C_100n_0402 C27
 U 1 1 6245FC31
 P 1700 1500
-F 0 "C?" H 1815 1545 60  0000 L CNN
+F 0 "C27" H 1815 1545 60  0000 L CNN
 F 1 "C_100n_0402" H 1700 1350 60  0001 C CNN
 F 2 "antmicro-footprints:0402-cap" H 1900 1700 60  0001 L CNN
@@
 $EndComp
 $Comp
-L power:GND #PWR?
+L power:GND #PWR0334
 U 1 1 6246203F
 P 2250 1600
-F 0 "#PWR?" H 2250 1350 50  0001 C CNN
+F 0 "#PWR0334" H 2250 1350 50  0001 C CNN
 F 1 "GND" H 2255 1427 50  0000 C CNN
 F 2 "" H 2250 1600 50  0001 C CNN
@@
 	1700 1350 1700 1200
 $Comp
-L power:GND #PWR?
+L power:GND #PWR0335
 U 1 1 6246365B
 P 1700 1700
-F 0 "#PWR?" H 1700 1450 50  0001 C CNN
+F 0 "#PWR0335" H 1700 1450 50  0001 C CNN
 F 1 "GND" H 1705 1527 50  0000 C CNN
 F 2 "" H 1700 1700 50  0001 C CNN
@@
 	1700 1700 1700 1650
 $Comp
-L antmicroCapacitors0402:C_100n_0402 C?
+L antmicroCapacitors0402:C_100n_0402 C25
 U 1 1 62463CDF
 P 1300 1500
-F 0 "C?" H 1415 1545 60  0000 L CNN
+F 0 "C25" H 1415 1545 60  0000 L CNN
 F 1 "C_100n_0402" H 1300 1350 60  0001 C CNN
 F 2 "antmicro-footprints:0402-cap" H 1500 1700 60  0001 L CNN
@@
 	1300 1350 1300 1200
 $Comp
-L power:GND #PWR?
+L power:GND #PWR0336
 U 1 1 62463D3C
 P 1300 1700
-F 0 "#PWR?" H 1300 1450 50  0001 C CNN
+F 0 "#PWR0336" H 1300 1450 50  0001 C CNN
 F 1 "GND" H 1305 1527 50  0000 C CNN
 F 2 "" H 1300 1700 50  0001 C CNN
@@
 PS_3V3
 $Comp
-L power:GND #PWR?
+L power:GND #PWR0337
 U 1 1 62464C95
 P 2050 2350
-F 0 "#PWR?" H 2050 2100 50  0001 C CNN
+F 0 "#PWR0337" H 2050 2100 50  0001 C CNN
 F 1 "GND" H 2055 2177 50  0000 C CNN
 F 2 "" H 2050 2350 50  0001 C CNN
@@
 Connection ~ 1300 1200
 $Comp
-L antmicroResistors0402:R_100R_0402 R?
+L antmicroResistors0402:R_100R_0402 R15
 U 1 1 623F60B0
 P 3600 2400
-F 0 "R?" V 3555 2470 60  0000 L CNN
+F 0 "R15" V 3555 2470 60  0000 L CNN
 F 1 "R_100R_0402" H 3600 2250 60  0001 C CNN
 F 2 "antmicro-footprints:0402-res" H 3800 2600 60  0001 L CNN
@@
 $EndComp
 $Comp
-L antmicroResistors0402:R_100R_0402 R?
+L antmicroResistors0402:R_100R_0402 R12
 U 1 1 623FB342
 P 3600 1900
-F 0 "R?" V 3555 1970 60  0000 L CNN
+F 0 "R12" V 3555 1970 60  0000 L CNN
 F 1 "R_100R_0402" H 3600 1750 60  0001 C CNN
 F 2 "antmicro-footprints:0402-res" H 3800 2100 60  0001 L CNN
@@
 Connection ~ 3600 1700
 $Comp
-L antmicroOscillators:AX3DAF1-125.0000 Y?
+L antmicroOscillators:AX3DAF1-125.0000 Y4
 U 1 1 6240118C
 P 8650 5150
-F 0 "Y?" H 8675 5525 50  0000 C CNN
+F 0 "Y4" H 8675 5525 50  0000 C CNN
 F 1 "AX3DAF1-125.0000" H 8675 5434 50  0000 C CNN
 F 2 "antmicro-footprints:AX3DAF1" H 8900 4850 50  0001 C CNN
@@
 PS_3V3
 $Comp
-L antmicroResistors0402:R_100R_0402 R?
+L antmicroResistors0402:R_100R_0402 R98
 U 1 1 624017F6
 P 9250 5150
-F 0 "R?" V 9205 5220 60  0000 L CNN
+F 0 "R98" V 9205 5220 60  0000 L CNN
 F 1 "R_100R_0402" H 9250 5000 60  0001 C CNN
 F 2 "antmicro-footprints:0402-res" H 9450 5350 60  0001 L CNN
@@
 Connection ~ 9250 5350
 $Comp
-L power:GND #PWR?
+L power:GND #PWR0338
 U 1 1 62406B82
 P 8250 5400
-F 0 "#PWR?" H 8250 5150 50  0001 C CNN
+F 0 "#PWR0338" H 8250 5150 50  0001 C CNN
 F 1 "GND" H 8255 5227 50  0000 C CNN
 F 2 "" H 8250 5400 50  0001 C CNN
@@
 	8250 5300 8300 5300
 $Comp
-L antmicroCapacitors0402:C_100n_0402 C?
+L antmicroCapacitors0402:C_100n_0402 C198
 U 1 1 62407F72
 P 7450 5200
-F 0 "C?" H 7565 5245 60  0000 L CNN
+F 0 "C198" H 7565 5245 60  0000 L CNN
 F 1 "C_100n_0402" H 7450 5050 60  0001 C CNN
 F 2 "antmicro-footprints:0402-cap" H 7650 5400 60  0001 L CNN
@@
 $EndComp
 $Comp
-L power:GND #PWR?
+L power:GND #PWR0339
 U 1 1 6240805A
 P 7450 5400
-F 0 "#PWR?" H 7450 5150 50  0001 C CNN
+F 0 "#PWR0339" H 7450 5150 50  0001 C CNN
 F 1 "GND" H 7455 5227 50  0000 C CNN
 F 2 "" H 7450 5400 50  0001 C CNN
@@
 PS_CLK_EN
 $Comp
-L antmicroOscillators:XLL736027.000000X U?
+L antmicroOscillators:XLL736027.000000X U46
 U 1 1 626DB080
 P 8550 2000
-F 0 "U?" H 8600 2403 60  0000 C CNN
+F 0 "U46" H 8600 2403 60  0000 C CNN
 F 1 "XLL736027.000000X" H 8600 2297 60  0000 C CNN
 F 2 "antmicro-footprints:Oscillator_SMD_IDT_JU6-6_7.0x5.0mm_P2.54mm" H 8750 2200 60  0001 L CNN
@@
 $EndComp
 $Comp
-L antmicroResistors0402:R_100R_0402 R?
+L antmicroResistors0402:R_100R_0402 R99
 U 1 1 626DD55B
 P 9300 2050
-F 0 "R?" V 9255 2120 60  0000 L CNN
+F 0 "R99" V 9255 2120 60  0000 L CNN
 F 1 "R_100R_0402" H 9300 1900 60  0001 C CNN
 F 2 "antmicro-footprints:0402-res" H 9500 2250 60  0001 L CNN
@@
 PS_3V3
 $Comp
-L antmicroCapacitors0402:C_100n_0402 C?
+L antmicroCapacitors0402:C_100n_0402 C197
 U 1 1 626E4BD6
 P 7300 1950
-F 0 "C?" H 7415 1995 60  0000 L CNN
+F 0 "C197" H 7415 1995 60  0000 L CNN
 F 1 "C_100n_0402" H 7300 1800 60  0001 C CNN
 F 2 "antmicro-footprints:0402-cap" H 7500 2150 60  0001 L CNN
@@
 $EndComp
 $Comp
-L power:GND #PWR?
+L power:GND #PWR0340
 U 1 1 626E4BE0
 P 7300 2150
-F 0 "#PWR?" H 7300 1900 50  0001 C CNN
+F 0 "#PWR0340" H 7300 1900 50  0001 C CNN
 F 1 "GND" H 7305 1977 50  0000 C CNN
 F 2 "" H 7300 2150 50  0001 C CNN
@@
 	8550 1800 8550 1750
 $Comp
-L power:GND #PWR?
+L power:GND #PWR0341
 U 1 1 626E8668
 P 8550 2400
-F 0 "#PWR?" H 8550 2150 50  0001 C CNN
+F 0 "#PWR0341" H 8550 2150 50  0001 C CNN
 F 1 "GND" H 8555 2227 50  0000 C CNN
 F 2 "" H 8550 2400 50  0001 C CNN
@@
 DisplayPort GTH REFCLK: 27MHz LVDS
 $Comp
-L antmicroCrystals:ECS-2520MVLC-260-CM-TR Y?
+L antmicroCrystals:ECS-2520MVLC-260-CM-TR Y3
 U 1 1 6293B97C
 P 2150 6000
-F 0 "Y?" H 2594 6046 50  0000 L CNN
+F 0 "Y3" H 2594 6046 50  0000 L CNN
 F 1 "ECS-2520MVLC-260-CM-TR" H 900 6300 50  0000 L CNN
 F 2 "antmicro-footprints:Oscillator_SMD_ECS_2520MV-xxx-xx-4Pin_2.5x2.0mm" H 2600 5650 50  0001 C CNN
@@
 $EndComp
 $Comp
-L antmicroInterfaceDriversReceiversTransceivers:SN65LVDS1DR U?
+L antmicroInterfaceDriversReceiversTransceivers:SN65LVDS1DR U45
 U 1 1 6294621B
 P 3350 6000
-F 0 "U?" H 3500 6450 50  0000 C CNN
+F 0 "U45" H 3500 6450 50  0000 C CNN
 F 1 "SN65LVDS1DR" H 3700 6350 50  0000 C CNN
 F 2 "antmicro-footprints:SOIC-8_W3.9mm" H 3350 5550 50  0001 C CNN
@@
 $EndComp
 $Comp
-L antmicroCapacitors0402:C_100n_0402 C?
+L antmicroCapacitors0402:C_100n_0402 C28
 U 1 1 62973B73
 P 2300 5300
-F 0 "C?" H 2415 5345 60  0000 L CNN
+F 0 "C28" H 2415 5345 60  0000 L CNN
 F 1 "C_100n_0402" H 2300 5150 60  0001 C CNN
 F 2 "antmicro-footprints:0402-cap" H 2500 5500 60  0001 L CNN
@@
 $EndComp
 $Comp
-L antmicroCapacitors0402:C_100n_0402 C?
+L antmicroCapacitors0402:C_100n_0402 C29
 U 1 1 62974242
 P 2800 5300
-F 0 "C?" H 2915 5345 60  0000 L CNN
+F 0 "C29" H 2915 5345 60  0000 L CNN
 F 1 "C_100n_0402" H 2800 5150 60  0001 C CNN
 F 2 "antmicro-footprints:0402-cap" H 3000 5500 60  0001 L CNN
@@
 	2550 6000 2850 6000
 $Comp
-L power:GND #PWR?
+L power:GND #PWR0342
 U 1 1 6297A7C2
 P 2150 6400
-F 0 "#PWR?" H 2150 6150 50  0001 C CNN
+F 0 "#PWR0342" H 2150 6150 50  0001 C CNN
 F 1 "GND" H 2155 6227 50  0000 C CNN
 F 2 "" H 2150 6400 50  0001 C CNN
@@
 	2150 6400 2150 6300
 $Comp
-L power:GND #PWR?
+L power:GND #PWR0343
 U 1 1 6297D3F9
 P 3350 6500
-F 0 "#PWR?" H 3350 6250 50  0001 C CNN
+F 0 "#PWR0343" H 3350 6250 50  0001 C CNN
 F 1 "GND" H 3355 6327 50  0000 C CNN
 F 2 "" H 3350 6500 50  0001 C CNN
@@
 	3350 6500 3350 6400
 $Comp
-L antmicroResistors0402:R_100R_0402 R?
+L antmicroResistors0402:R_100R_0402 R16
 U 1 1 6298446A
 P 4100 6000
-F 0 "R?" V 4055 6070 60  0000 L CNN
+F 0 "R16" V 4055 6070 60  0000 L CNN
 F 1 "R_100R_0402" H 4100 5850 60  0001 C CNN
 F 2 "antmicro-footprints:0402-res" H 4300 6200 60  0001 L CNN
@@
 GTR_REFCLK0_C2M_N
 $Comp
-L power:GND #PWR?
+L power:GND #PWR0344
 U 1 1 6298F9EC
 P 2300 5550
-F 0 "#PWR?" H 2300 5300 50  0001 C CNN
+F 0 "#PWR0344" H 2300 5300 50  0001 C CNN
 F 1 "GND" H 2305 5377 50  0000 C CNN
 F 2 "" H 2300 5550 50  0001 C CNN
@@
 $EndComp
 $Comp
-L power:GND #PWR?
+L power:GND #PWR0345
 U 1 1 62995216
 P 2800 5550
-F 0 "#PWR?" H 2800 5300 50  0001 C CNN
+F 0 "#PWR0345" H 2800 5300 50  0001 C CNN
 F 1 "GND" H 2805 5377 50  0000 C CNN
 F 2 "" H 2800 5550 50  0001 C CNN

Commit message: fixed an issue with reset logic (Mixed PS and PL domain on OD buffer), extended the logic circuit to support M.2 PERST# (reset for PCIe WIFI), fixed the polarity of the camera control signal CAM_RST to comply with Antmicro standard, change CAM _SHDN to CAM_VSYNC, replaced the reset connector to fit additional signal M2_PERST
Parts:
- removed C25, C27: C_100n_0402, antmicro-footprints:0402-cap, symbol antmicroCapacitors0402:C_100n_0402
- removed U2: DSC557-0333FI1, antmicro-footprints:MICROCHIP_QFN14_3.2X2.5, symbol antmicroClockTimingRealTimeClocks:DSC557-0333FI1
- added C? (x5): C_100n_0402, antmicro-footprints:0402-cap, symbol antmicroCapacitors0402:C_100n_0402
- added Q?: BSS138-7-F, antmicro-footprints:SOT-23-3, symbol antmicroTransistorsFETsMOSFETsSingle:BSS138-7-F
- added R?: R_100R_0402, antmicro-footprints:0402-res, symbol antmicroResistors0402:R_100R_0402
- added R?: R_10k_0402, antmicro-footprints:0402-res, symbol antmicroResistors0402:R_10k_0402
- added R?: R_1M0_0402, antmicro-footprints:0402-res, symbol antmicroResistors0402:R_1M0_0402
- added U?: SI53152-A01AGMR, antmicro-footprints:SIL_QFN24_4X4, symbol antmicroLogicBuffersDriversReceiversTransceivers:SI53152-A01AGMR
- added Y?: SIT9120AI-2C3-33E100.000000X, antmicro-footprints:SiTime_5.0x3.2, symbol antmicroOscillators:SIT9120AI-2C3-33E100.000000X
Connections:
- net labels added: ~M2_CLKREQ
- wire segments 90 -> 142
- no-connect marks 0 -> 2
Other:
- moved on the sheet: C197, C198, C28, C29, R12, R15, R16, R98, R99, U45, U46, Y3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
