File: kria-k26-devboard/usbc-socket.sch (KiCad schematic (older format))
At the start: 8 parts, among them J10 USB4105-GF-A, Q15 PJA3441, Q16 BSS138-7-F

Commit message: Routed I2C, JTAG, PS reset, remaining differential pairs. Component optimization
Parts:
- added U53: WE-TVS-82400152, antmicro-footprints:SOT-563, symbol antmicroTVSDiodes:WE-TVS-82400152
Changed lines of the file:
@@
 Wire Wire Line
 	6300 3150 6300 3100
-Wire Bus Line
-	6500 3350 6500 3550
 $Comp
 L antmicroUSBDVIHDMIConnectors:USB4105-GF-A J?
@@
 	1    0    0    -1
 $EndComp
+$Comp
+L antmicroTVSDiodes:WE-TVS-82400152 U?
+U 1 1 62E99410
+P 5150 5750
+AR Path="/625B0244/62E99410" Ref="U?"  Part="1"
+AR Path="/63C44BC2/62A9ECDC/62E99410" Ref="U53"  Part="1"
+F 0 "U53" H 5100 5950 50  0000 R CNN
+F 1 "WE-TVS-82400152" H 5550 5550 50  0000 R CNN
+F 2 "antmicro-footprints:SOT-563" H 5150 5550 50  0001 C CNN
+F 3 "https://katalog.we-online.de/pbs/datasheet/82400102.pdf" H 5150 5500 50  0001 C CNN
+F 4 "82400152" H 4800 5350 50  0001 C CNN "MPN"
+F 5 "Würth Elektronik" H 4900 5450 50  0001 C CNN "Manufacturer"
+	1    5150 5750
+	0    -1   -1   0
+$EndComp
+Wire Bus Line
+	6500 3350 6500 3550
 $EndSCHEMATC

Commit message: Routed USB debug part, DP AUX, Supply for SD 3.0, improved decoupling. Other minor improvments
Connections:
- wire segments 61 -> 64
Changed lines of the file:
@@
 	4450 4600 4600 4600
 Wire Wire Line
-	4500 4150 4450 4150
-Wire Wire Line
-	4450 4050 4500 4050
-Wire Wire Line
-	4500 3900 4450 3900
-Wire Wire Line
-	4450 3800 4500 3800
-Text Label 4900 3650 2    50   ~ 0
-USBC_CC2
-Text Label 4900 3550 2    50   ~ 0
-USBC_CC1
+	4500 4100 4450 4100
+Wire Wire Line
+	4450 4000 4500 4000
+Wire Wire Line
+	4500 3850 4450 3850
+Wire Wire Line
+	4450 3750 4500 3750
 $Comp
 L antmicroTVSDiodes:ESD144B1W0201E6327XTSA1 D?
@@
 	0    1    1    0
 $EndComp
-Text Label 4500 3350 0    50   ~ 0
-USBC_VBUS
 $Comp
 L power:GND #PWR?
@@
 	1    0    0    -1
 $EndComp
-Text HLabel 6650 3350 2    50   Input ~ 0
+Text HLabel 6650 3300 2    50   Input ~ 0
 USBC_CC[1..2]
 Wire Bus Line
-	6650 3350 6500 3350
+	6650 3300 6500 3300
 NoConn ~ 4450 4400
 NoConn ~ 4450 4300
@@
 $Comp
 L antmicroTVSDiodes:PESD2USB5UV-TR D?
-U 1 1 62AA36AF
-P 6450 4500
-AR Path="/63C44BC2/62AA36AF" Ref="D?"  Part="1"
-AR Path="/63C44BC2/62A9ECDC/62AA36AF" Ref="D27"  Part="1"
-F 0 "D27" H 6450 4650 60  0000 L CNN
-F 1 "PESD2USB5UV-TR" H 6300 4150 60  0000 L CNN
-F 2 "antmicro-footprints:SOT-23s" H 6500 4700 60  0001 C CNN
-F 3 "https://assets.nexperia.com/documents/data-sheet/PESD2USB5UV-T.pdf" H 6450 4500 60  0001 C CNN
-F 4 "PESD2USB5UV-TR " H 6150 4800 50  0001 C CNN "MPN"
-F 5 "Nexperia " H 6150 4900 50  0001 C CNN "Manufacturer"
-	1    6450 4500
-	1    0    0    -1
-$EndComp
-$Comp
-L power:GND #PWR?
-U 1 1 62AA36B9
-P 6200 4750
-AR Path="/63C44BC2/62AA36B9" Ref="#PWR?"  Part="1"
-AR Path="/63C44BC2/62A9ECDC/62AA36B9" Ref="#PWR0377"  Part="1"
-F 0 "#PWR0377" H 6200 4500 50  0001 C CNN
-F 1 "GND" H 6205 4577 50  0000 C CNN
-F 2 "" H 6200 4750 50  0001 C CNN
-F 3 "" H 6200 4750 50  0001 C CNN
-	1    6200 4750
-	1    0    0    -1
-$EndComp
-Wire Wire Line
-	6200 4750 6200 4700
-Wire Wire Line
-	6200 4700 6250 4700
-Wire Wire Line
-	6250 4500 6200 4500
-Wire Wire Line
-	6250 4600 6100 4600
-$Comp
-L antmicroTVSDiodes:PESD2USB5UV-TR D?
 U 1 1 62AA36C7
 P 5400 4500
@@
 Wire Wire Line
 	5200 4600 5050 4600
-Wire Wire Line
-	5050 4600 5050 3650
-Connection ~ 5050 3650
-Wire Wire Line
-	5050 3650 4450 3650
 Text HLabel 5000 2200 1    50   Output ~ 0
 USBC_VBUS
@@
 Connection ~ 5600 2250
 Entry Wire Line
-	6500 3550 6400 3650
+	6500 3500 6400 3600
 Entry Wire Line
-	6500 3450 6400 3550
+	6500 3400 6400 3500
+Wire Wire Line
+	4500 4000 4500 4050
+Wire Wire Line
+	4500 3750 4500 3800
+Wire Wire Line
+	4500 3800 4750 3800
+Wire Wire Line
+	4750 3800 4750 3900
+Wire Wire Line
+	6550 3900 6550 3850
+Wire Wire Line
+	6550 3850 6600 3850
+Connection ~ 4500 3800
+Wire Wire Line
+	4500 3800 4500 3850
+Wire Wire Line
+	4500 4050 4750 4050
+Wire Wire Line
+	4750 4050 4750 3950
+Wire Wire Line
+	6550 3950 6550 4000
+Wire Wire Line
+	6550 4000 6600 4000
+Connection ~ 4500 4050
 Wire Wire Line
 	4500 4050 4500 4100
-Wire Wire Line
-	4500 3800 4500 3850
-Wire Wire Line
-	4500 3850 4750 3850
-Wire Wire Line
-	4750 3850 4750 3950
-Wire Wire Line
-	6550 3950 6550 3900
-Wire Wire Line
-	6550 3900 6600 3900
-Connection ~ 4500 3850
-Wire Wire Line
-	4500 3850 4500 3900
-Wire Wire Line
-	4500 4100 4750 4100
-Wire Wire Line
-	4750 4100 4750 4000
-Wire Wire Line
-	6550 4000 6550 4050
-Wire Wire Line
-	6550 4050 6600 4050
-Connection ~ 4500 4100
-Wire Wire Line
-	4500 4100 4500 4150
-Text HLabel 6600 3900 2    50   Input ~ 0
+Text HLabel 6600 3850 2    50   Input ~ 0
 USBC_P
-Text HLabel 6600 4050 2    50   Input ~ 0
+Text HLabel 6600 4000 2    50   Input ~ 0
 USBC_N
 Wire Wire Line
-	6100 3950 6100 4600
-Wire Wire Line
-	6100 3950 6550 3950
-Wire Wire Line
-	6200 4000 6550 4000
-Wire Wire Line
-	6200 4000 6200 4500
-Connection ~ 6200 4000
-Wire Wire Line
-	4750 4000 6200 4000
-Connection ~ 6100 3950
-Wire Wire Line
-	4750 3950 6100 3950
-Wire Wire Line
-	4450 3350 5000 3350
+	6100 3900 6550 3900
+Wire Wire Line
+	6200 3950 6550 3950
+Connection ~ 6200 3950
+Wire Wire Line
+	4750 3950 6200 3950
+Connection ~ 6100 3900
+Wire Wire Line
+	4750 3900 6100 3900
 Wire Wire Line
 	5000 2250 5250 2250
 Wire Wire Line
-	5000 2250 5000 3350
+	5000 2250 5000 3250
 Connection ~ 5250 2250
 $Comp
@@
 $EndComp
 Wire Wire Line
-	5050 3650 6400 3650
-Wire Wire Line
-	4450 3550 5150 3550
-Wire Wire Line
-	5150 3550 5150 4500
-Connection ~ 5150 3550
-Wire Wire Line
-	5150 3550 6400 3550
+	5050 3600 6400 3600
+Wire Wire Line
+	5150 3500 6400 3500
 Wire Wire Line
 	5000 2250 5000 2200
@@
 	0    -1   -1   0
 $EndComp
+Text Label 4900 3600 2    50   ~ 0
+USBC_CC2
+Text Label 4900 3500 2    50   ~ 0
+USBC_CC1
+Connection ~ 5050 3600
+Wire Wire Line
+	5050 3600 4450 3600
+Connection ~ 5150 3500
+Wire Wire Line
+	4450 3500 5150 3500
+Wire Wire Line
+	6200 4750 6200 4700
+Wire Wire Line
+	6250 4600 6100 4600
+Wire Wire Line
+	6250 4500 6200 4500
+Wire Wire Line
+	6200 4700 6250 4700
+$Comp
+L power:GND #PWR?
+U 1 1 62AA36B9
+P 6200 4750
+AR Path="/63C44BC2/62AA36B9" Ref="#PWR?"  Part="1"
+AR Path="/63C44BC2/62A9ECDC/62AA36B9" Ref="#PWR0377"  Part="1"
+F 0 "#PWR0377" H 6200 4500 50  0001 C CNN
+F 1 "GND" H 6205 4577 50  0000 C CNN
+F 2 "" H 6200 4750 50  0001 C CNN
+F 3 "" H 6200 4750 50  0001 C CNN
+	1    6200 4750
+	1    0    0    -1
+$EndComp
+$Comp
+L antmicroTVSDiodes:PESD2USB5UV-TR D?
+U 1 1 62AA36AF
+P 6450 4500
+AR Path="/63C44BC2/62AA36AF" Ref="D?"  Part="1"
+AR Path="/63C44BC2/62A9ECDC/62AA36AF" Ref="D27"  Part="1"
+F 0 "D27" H 6450 4650 60  0000 L CNN
+F 1 "PESD2USB5UV-TR" H 6300 4150 60  0000 L CNN
+F 2 "antmicro-footprints:SOT-23s" H 6500 4700 60  0001 C CNN
+F 3 "https://assets.nexperia.com/documents/data-sheet/PESD2USB5UV-T.pdf" H 6450 4500 60  0001 C CNN
+F 4 "PESD2USB5UV-TR " H 6150 4800 50  0001 C CNN "MPN"
+F 5 "Nexperia " H 6150 4900 50  0001 C CNN "Manufacturer"
+	1    6450 4500
+	1    0    0    -1
+$EndComp
+Wire Wire Line
+	6100 3900 6100 4600
+Wire Wire Line
+	6200 3950 6200 4500
+Wire Wire Line
+	5150 3500 5150 4500
+Wire Wire Line
+	5050 3600 5050 4600
+Wire Wire Line
+	4450 3350 4500 3350
+Wire Wire Line
+	4500 3350 4500 3250
+Wire Wire Line
+	4500 3250 4450 3250
+Wire Wire Line
+	4500 3250 5000 3250
+Connection ~ 4500 3250
 Wire Bus Line
-	6500 3350 6500 3550
+	6500 3300 6500 3500
 $EndSCHEMATC

Commit message: Removed PL_1V2 DC-DC, Routed: signalling voltage selector for SD 3.0, reset signals and DC-DC enables, VSYNC, ETH connector diff. pairs, missing USB 3.0 diff. pair. Created planes for PoE adnd DC_MAIN_BUS
Parts:
- removed Q16: BSS138-7-F, antmicro-footprints:SOT-23-3, symbol antmicroTransistorsFETsMOSFETsSingle:BSS138-7-F
- added Q11: DTC014TEBTL, antmicro-footprints:SOT-416, symbol antmicroTransistorsBipolarSingle:DTC014TEBTL
Changed lines of the file:
@@
 Wire Wire Line
 	6300 2650 6300 2550
-Text HLabel 6650 3000 2    50   Input ~ 0
+Text HLabel 6700 2900 2    50   Input ~ 0
 PD_EN
 Wire Wire Line
-	6650 3000 6600 3000
-$Comp
-L antmicroTransistorsFETsMOSFETsSingle:BSS138-7-F Q16
-U 1 1 661CFCBB
-P 6300 2900
-F 0 "Q16" H 6407 2953 60  0000 L CNN
-F 1 "BSS138-7-F" V 6550 2450 60  0000 L CNN
-F 2 "antmicro-footprints:SOT-23-3" H 6500 3100 60  0001 L CNN
-F 3 "https://www.diodes.com/assets/Datasheets/ds30144.pdf" H 6500 3200 60  0001 L CNN
-F 4 "BSS138-7-F" H 6500 3400 60  0001 L CNN "MPN"
-F 5 "Diodes Incorporated" H 6500 4000 60  0001 L CNN "Manufacturer"
-	1    6300 2900
-	-1   0    0    -1
-$EndComp
+	6700 2900 6650 2900
 Wire Wire Line
 	6300 2700 6300 2650
@@
 	4500 3250 5000 3250
 Connection ~ 4500 3250
+$Comp
+L antmicroTransistorsBipolarSingle:DTC014TEBTL Q11
+U 1 1 631791E8
+P 6400 2900
+F 0 "Q11" H 6588 2946 50  0000 L CNN
+F 1 "DTC014TEBTL" H 5950 3100 50  0000 L CNN
+F 2 "antmicro-footprints:SOT-416" H 6600 2600 50  0001 L CNN
+F 3 "" H 6400 2900 50  0001 L CNN
+F 4 "ROHM Semiconductor" H 7000 2800 50  0001 C CNN "Manufacturer"
+F 5 "DTC014TEBTL" H 6850 2700 50  0001 C CNN "MPN"
+	1    6400 2900
+	-1   0    0    -1
+$EndComp
 Wire Bus Line
 	6500 3300 6500 3500

Commit message: Replaced PCIe clock generation (LVDS to HCSL), Clock component size optimization for USB, Optimized ESD protection for PD USB, placed and routed new clock circuitry, clock signals recalculated to 100Ohm  and re-routed
Parts:
- removed D25, D27: PESD2USB5UV-TR, antmicro-footprints:SOT-23s, symbol antmicroTVSDiodes:PESD2USB5UV-TR
- removed D26: ESD144B1W0201E6327XTSA1, antmicro-footprints:ESD144B1W0201E6327XTSA1, symbol antmicroTVSDiodes:ESD144B1W0201E6327XTSA1
- added D1: SMF4L15CA, antmicro-footprints:SOD-123FL, symbol antmicroTVSDiodes:SMF4L15CA
- added U56: WE-TVS-82400152, antmicro-footprints:SOT-563, symbol antmicroTVSDiodes:WE-TVS-82400152
Connections:
- net labels added: USBC_TVS_CC1, USBC_TVS_CC2, USBC_TVS_N, USBC_TVS_P
- wire segments 64 -> 70
- no-connect marks 2 -> 4
Other:
- moved on the sheet: U53
Changed lines of the file:
@@
 	4450 3750 4500 3750
-$Comp
-L antmicroTVSDiodes:ESD144B1W0201E6327XTSA1 D?
-U 1 1 62AA3683
-P 5600 2650
-AR Path="/63C44BC2/62AA3683" Ref="D?"  Part="1"
-AR Path="/63C44BC2/62A9ECDC/62AA3683" Ref="D26"  Part="1"
-F 0 "D26" V 5554 2728 50  0000 L CNN
-F 1 "ESD144B1W0201E6327XTSA1" H 5250 2900 50  0000 L CNN
-F 2 "antmicro-footprints:ESD144B1W0201E6327XTSA1" H 5600 2650 50  0001 C CNN
-F 3 "https://www.infineon.com/dgdl/Infineon-ESD144-B1-W0201-DataSheet-v02_00-EN.pdf?fileId=5546d462677d0f4601679886a2a8707c" H 5600 2650 50  0001 C CNN
-F 4 "ESD144B1W0201E6327XTSA1" H 5600 2650 50  0001 C CNN "MPN"
-F 5 "Infineon Technologies" H 5600 2650 50  0001 C CNN "Manufacturer"
-	1    5600 2650
-	0    1    1    0
-$EndComp
 $Comp
 L power:GND #PWR?
@@
 	1    0    0    -1
 $EndComp
-Text HLabel 6650 3300 2    50   Input ~ 0
+Text HLabel 6850 3450 2    50   Input ~ 0
 USBC_CC[1..2]
 Wire Bus Line
-	6650 3300 6500 3300
-NoConn ~ 4450 4400
-NoConn ~ 4450 4300
+	6850 3450 6700 3450
+NoConn ~ 4450 4350
+NoConn ~ 4450 4250
 $Comp
 L antmicroCapacitorsmisc:C_100n_0402_50V C?
@@
 Wire Wire Line
 	5600 3050 5600 3150
-$Comp
-L antmicroTVSDiodes:PESD2USB5UV-TR D?
-U 1 1 62AA36C7
-P 5400 4500
-AR Path="/63C44BC2/62AA36C7" Ref="D?"  Part="1"
-AR Path="/63C44BC2/62A9ECDC/62AA36C7" Ref="D25"  Part="1"
-F 0 "D25" H 5400 4700 60  0000 L CNN
-F 1 "PESD2USB5UV-TR" H 5250 4150 60  0000 L CNN
-F 2 "antmicro-footprints:SOT-23s" H 5450 4700 60  0001 C CNN
-F 3 "https://assets.nexperia.com/documents/data-sheet/PESD2USB5UV-T.pdf" H 5400 4500 60  0001 C CNN
-F 4 "PESD2USB5UV-TR " H 5100 4800 50  0001 C CNN "MPN"
-F 5 "Nexperia " H 5100 4900 50  0001 C CNN "Manufacturer"
-	1    5400 4500
-	1    0    0    -1
-$EndComp
-$Comp
-L power:GND #PWR?
-U 1 1 62AA36CD
-P 5150 4750
-AR Path="/63C44BC2/62AA36CD" Ref="#PWR?"  Part="1"
-AR Path="/63C44BC2/62A9ECDC/62AA36CD" Ref="#PWR0375"  Part="1"
-F 0 "#PWR0375" H 5150 4500 50  0001 C CNN
-F 1 "GND" H 5155 4577 50  0000 C CNN
-F 2 "" H 5150 4750 50  0001 C CNN
-F 3 "" H 5150 4750 50  0001 C CNN
-	1    5150 4750
-	1    0    0    -1
-$EndComp
-Wire Wire Line
-	5150 4750 5150 4700
-Wire Wire Line
-	5150 4700 5200 4700
-Wire Wire Line
-	5200 4500 5150 4500
-Wire Wire Line
-	5200 4600 5050 4600
 Text HLabel 5000 2200 1    50   Output ~ 0
 USBC_VBUS
@@
 Connection ~ 5600 2250
 Entry Wire Line
-	6500 3500 6400 3600
+	6700 3750 6600 3850
 Entry Wire Line
-	6500 3400 6400 3500
+	6700 3550 6600 3650
 Wire Wire Line
 	4500 4000 4500 4050
@@
 	4500 3750 4500 3800
 Wire Wire Line
-	4500 3800 4750 3800
-Wire Wire Line
-	4750 3800 4750 3900
-Wire Wire Line
-	6550 3900 6550 3850
-Wire Wire Line
-	6550 3850 6600 3850
+	4500 3800 4550 3800
 Connection ~ 4500 3800
 Wire Wire Line
 	4500 3800 4500 3850
 Wire Wire Line
-	4500 4050 4750 4050
-Wire Wire Line
-	4750 4050 4750 3950
-Wire Wire Line
-	6550 3950 6550 4000
-Wire Wire Line
-	6550 4000 6600 4000
+	6700 4450 6800 4450
 Connection ~ 4500 4050
 Wire Wire Line
 	4500 4050 4500 4100
-Text HLabel 6600 3850 2    50   Input ~ 0
+Text HLabel 6800 4350 2    50   Input ~ 0
 USBC_P
-Text HLabel 6600 4000 2    50   Input ~ 0
+Text HLabel 6800 4450 2    50   Input ~ 0
 USBC_N
-Wire Wire Line
-	6100 3900 6550 3900
-Wire Wire Line
-	6200 3950 6550 3950
-Connection ~ 6200 3950
-Wire Wire Line
-	4750 3950 6200 3950
-Connection ~ 6100 3900
-Wire Wire Line
-	4750 3900 6100 3900
 Wire Wire Line
 	5000 2250 5250 2250
@@
 	0    1    -1   0
 $EndComp
-Wire Wire Line
-	5050 3600 6400 3600
-Wire Wire Line
-	5150 3500 6400 3500
 Wire Wire Line
 	5000 2250 5000 2200
@@
 	1    0    0    -1
 $EndComp
-$Comp
-L antmicroTVSDiodes:WE-TVS-82400152 U?
-U 1 1 62E99410
-P 5150 5750
-AR Path="/625B0244/62E99410" Ref="U?"  Part="1"
-AR Path="/63C44BC2/62A9ECDC/62E99410" Ref="U53"  Part="1"
-F 0 "U53" H 5100 5950 50  0000 R CNN
-F 1 "WE-TVS-82400152" H 5550 5550 50  0000 R CNN
-F 2 "antmicro-footprints:SOT-563" H 5150 5550 50  0001 C CNN
-F 3 "https://katalog.we-online.de/pbs/datasheet/82400102.pdf" H 5150 5500 50  0001 C CNN
-F 4 "82400152" H 4800 5350 50  0001 C CNN "MPN"
-F 5 "Würth Elektronik" H 4900 5450 50  0001 C CNN "Manufacturer"
-	1    5150 5750
-	0    -1   -1   0
-$EndComp
-Text Label 4900 3600 2    50   ~ 0
+Text Label 6550 3850 2    50   ~ 0
 USBC_CC2
-Text Label 4900 3500 2    50   ~ 0
+Text Label 6550 3650 2    50   ~ 0
 USBC_CC1
-Connection ~ 5050 3600
-Wire Wire Line
-	5050 3600 4450 3600
-Connection ~ 5150 3500
-Wire Wire Line
-	4450 3500 5150 3500
-Wire Wire Line
-	6200 4750 6200 4700
-Wire Wire Line
-	6250 4600 6100 4600
-Wire Wire Line
-	6250 4500 6200 4500
-Wire Wire Line
-	6200 4700 6250 4700
-$Comp
-L power:GND #PWR?
-U 1 1 62AA36B9
-P 6200 4750
-AR Path="/63C44BC2/62AA36B9" Ref="#PWR?"  Part="1"
-AR Path="/63C44BC2/62A9ECDC/62AA36B9" Ref="#PWR0377"  Part="1"
-F 0 "#PWR0377" H 6200 4500 50  0001 C CNN
-F 1 "GND" H 6205 4577 50  0000 C CNN
-F 2 "" H 6200 4750 50  0001 C CNN
-F 3 "" H 6200 4750 50  0001 C CNN
-	1    6200 4750
-	1    0    0    -1
-$EndComp
-$Comp
-L antmicroTVSDiodes:PESD2USB5UV-TR D?
-U 1 1 62AA36AF
-P 6450 4500
-AR Path="/63C44BC2/62AA36AF" Ref="D?"  Part="1"
-AR Path="/63C44BC2/62A9ECDC/62AA36AF" Ref="D27"  Part="1"
-F 0 "D27" H 6450 4650 60  0000 L CNN
-F 1 "PESD2USB5UV-TR" H 6300 4150 60  0000 L CNN
-F 2 "antmicro-footprints:SOT-23s" H 6500 4700 60  0001 C CNN
-F 3 "https://assets.nexperia.com/documents/data-sheet/PESD2USB5UV-T.pdf" H 6450 4500 60  0001 C CNN
-F 4 "PESD2USB5UV-TR " H 6150 4800 50  0001 C CNN "MPN"
-F 5 "Nexperia " H 6150 4900 50  0001 C CNN "Manufacturer"
-	1    6450 4500
-	1    0    0    -1
-$EndComp
-Wire Wire Line
-	6100 3900 6100 4600
-Wire Wire Line
-	6200 3950 6200 4500
-Wire Wire Line
-	5150 3500 5150 4500
-Wire Wire Line
-	5050 3600 5050 4600
 Wire Wire Line
 	4450 3350 4500 3350
@@
 	-1   0    0    -1
 $EndComp
+$Comp
+L antmicroTVSDiodes:WE-TVS-82400152 U?
+U 1 1 62E99410
+P 5850 4400
+AR Path="/625B0244/62E99410" Ref="U?"  Part="1"
+AR Path="/63C44BC2/62A9ECDC/62E99410" Ref="U53"  Part="1"
+F 0 "U53" H 5800 4600 50  0000 R CNN
+F 1 "WE-TVS-82400152" H 6250 4200 50  0000 R CNN
+F 2 "antmicro-footprints:SOT-563" H 5850 4200 50  0001 C CNN
+F 3 "https://katalog.we-online.de/pbs/datasheet/82400102.pdf" H 5850 4150 50  0001 C CNN
+F 4 "82400152" H 5500 4000 50  0001 C CNN "MPN"
+F 5 "Würth Elektronik" H 5600 4100 50  0001 C CNN "Manufacturer"
+	1    5850 4400
+	-1   0    0    1
+$EndComp
+Wire Wire Line
+	4500 4050 4550 4050
+NoConn ~ 5550 4400
+$Comp
+L power:GND #PWR?
+U 1 1 63812C2B
+P 6550 4550
+AR Path="/63C44BC2/63812C2B" Ref="#PWR?"  Part="1"
+AR Path="/63C44BC2/62A9ECDC/63812C2B" Ref="#PWR0375"  Part="1"
+F 0 "#PWR0375" H 6550 4300 50  0001 C CNN
+F 1 "GND" H 6555 4377 50  0000 C CNN
+F 2 "" H 6550 4550 50  0001 C CNN
+F 3 "" H 6550 4550 50  0001 C CNN
+	1    6550 4550
+	1    0    0    -1
+$EndComp
+Wire Wire Line
+	6550 4400 6150 4400
+Wire Wire Line
+	6550 4400 6550 4550
+Wire Wire Line
+	6150 4500 6700 4500
+Wire Wire Line
+	6700 4500 6700 4450
+Wire Wire Line
+	6150 4300 6700 4300
+Wire Wire Line
+	6700 4300 6700 4350
+Wire Wire Line
+	6700 4350 6800 4350
+Text Label 4550 3900 0    50   ~ 0
+USBC_TVS_P
+Wire Wire Line
+	4550 3800 4550 3900
+Wire Wire Line
+	4550 3900 5200 3900
+Wire Wire Line
+	4550 4050 4550 4000
+Text Label 4550 4000 0    50   ~ 0
+USBC_TVS_N
+Text Label 5100 3500 2    50   ~ 0
+USBC_TVS_CC1
+Text Label 5100 3600 2    50   ~ 0
+USBC_TVS_CC2
+$Comp
+L antmicroTVSDiodes:WE-TVS-82400152 U?
+U 1 1 6383DAA4
+P 5800 3750
+AR Path="/625B0244/6383DAA4" Ref="U?"  Part="1"
+AR Path="/63C44BC2/62A9ECDC/6383DAA4" Ref="U56"  Part="1"
+F 0 "U56" H 5750 3950 50  0000 R CNN
+F 1 "WE-TVS-82400152" H 6200 3550 50  0000 R CNN
+F 2 "antmicro-footprints:SOT-563" H 5800 3550 50  0001 C CNN
+F 3 "https://katalog.we-online.de/pbs/datasheet/82400102.pdf" H 5800 3500 50  0001 C CNN
+F 4 "82400152" H 5450 3350 50  0001 C CNN "MPN"
+F 5 "Würth Elektronik" H 5550 3450 50  0001 C CNN "Manufacturer"
+	1    5800 3750
+	-1   0    0    1
+$EndComp
+Wire Wire Line
+	6100 3850 6600 3850
+Wire Wire Line
+	6100 3650 6600 3650
+$Comp
+L power:GND #PWR?
+U 1 1 6386B45F
+P 6150 3900
+AR Path="/63C44BC2/6386B45F" Ref="#PWR?"  Part="1"
+AR Path="/63C44BC2/62A9ECDC/6386B45F" Ref="#PWR0377"  Part="1"
+F 0 "#PWR0377" H 6150 3650 50  0001 C CNN
+F 1 "GND" H 6155 3727 50  0000 C CNN
+F 2 "" H 6150 3900 50  0001 C CNN
+F 3 "" H 6150 3900 50  0001 C CNN
+	1    6150 3900
+	1    0    0    -1
+$EndComp
+Wire Wire Line
+	6150 3750 6150 3900
+Wire Wire Line
+	6150 3750 6100 3750
+NoConn ~ 5500 3750
+Wire Wire Line
+	5150 4000 5150 4450
+Wire Wire Line
+	4550 4000 5150 4000
+Wire Wire Line
+	5250 3600 5250 3850
+Wire Wire Line
+	5250 3850 5500 3850
+Wire Wire Line
+	4450 3600 5250 3600
+Wire Wire Line
+	5500 3650 5300 3650
+Wire Wire Line
+	5300 3650 5300 3500
+Wire Wire Line
+	4450 3500 5300 3500
+Wire Wire Line
+	5200 4350 5500 4350
+Wire Wire Line
+	5500 4350 5500 4300
+Wire Wire Line
+	5500 4300 5550 4300
+Wire Wire Line
+	5500 4500 5500 4450
+Wire Wire Line
+	5500 4500 5550 4500
+Wire Wire Line
+	5200 3900 5200 4350
+Wire Wire Line
+	4450 4500 4600 4500
+Wire Wire Line
+	4600 4500 4600 4600
+Wire Wire Line
+	5150 4450 5500 4450
+Connection ~ 4600 4600
+$Comp
+L antmicroTVSDiodes:SMF4L15CA D1
+U 1 1 626860F1
+P 5600 2650
+F 0 "D1" V 5554 2728 50  0000 L CNN
+F 1 "SMF4L15CA" V 5645 2728 50  0000 L CNN
+F 2 "antmicro-footprints:SOD-123FL" H 5600 2650 50  0001 C CNN
+F 3 "https://www.mouser.pl/datasheet/2/240/Littelfuse_TVS_Diode_SMF4L_Datasheet_pdf-1665786.pdf" H 5600 2650 50  0001 C CNN
+F 4 "SMF4L15CA" H 5600 2650 50  0001 C CNN "MPN"
+F 5 "Infineon Technologies" H 5600 2650 50  0001 C CNN "Manufacturer"
+	1    5600 2650
+	0    1    1    0
+$EndComp
 Wire Bus Line
-	6500 3300 6500 3500
+	6700 3450 6700 3750
 $EndSCHEMATC
