File: dc-dc-conventers.sch (KiCad schematic (older format))
At the start: 113 parts, among them Q13 DTC014TEBTL, Q14 DTC014TEBTL, Q15 DTC014TEBTL, U47 RT6236AHGQUF, U48 RT6236AHGQUF, U49 AP62301WU-7, U50 AP62301WU-7, U51 AP62301WU-7, U52 AP62301WU-7, U53 AP62301WU-7, U54 AP62301WU-7, U55 AP62301WU-7

Commit message: Fixed wrong footprint assigment for L4 and L7, PCB changed to fit proper inductor footprints. Fixed R22 missing lib
Parts:
- removed L4, L7: TFM201208ALD-1R0MTCA, kria-k26-devboard-footprints:0603-res, symbol kria-k26-devboard:TFM201208ALD-1R0MTCA
- added L4, L7: TFM201208ALD-1R0MTCA, antmicro-footprints:0805-res, symbol antmicroFixedInductors:TFM201208ALD-1R0MTCA
Changed lines of the file:
@@
-	1    0    0    -1
-$EndComp
-$Comp
-L kria-k26-devboard:TFM201208ALD-1R0MTCA L4
-U 1 1 62B2FA71
-P 8850 2800
-F 0 "L4" H 8850 3105 60  0000 C CNN
-F 1 "TFM201208ALD-1R0MTCA" H 8850 2999 60  0000 C CNN
-F 2 "kria-k26-devboard-footprints:0603-res" H 9475 3150 60  0001 C CNN
-F 3 "https://product.tdk.com/system/files/dam/doc/product/inductor/inductor/smd/catalog/inductor_commercial_power_tfm201208ald_en.pdf" H 8905 2830 60  0001 C CNN
-F 4 "TDK" H 9000 3550 50  0001 C CNN "Manufacturer"
-F 5 "TFM201208ALD-1R0MTCA" H 9150 3450 50  0001 C CNN "MPN"
-F 6 "2.5A" H 8925 3350 50  0001 C CNN "MaxCur"
-F 7 "1.25x0.8" H 8975 3250 50  0001 C CNN "Size"
-F 8 "1u/2.5A" H 8850 2901 50  0000 C CNN "Val"
-	1    8850 2800
-	1    0    0    -1
-$EndComp
-$Comp
-L kria-k26-devboard:TFM201208ALD-1R0MTCA L7
-U 1 1 62B31FDC
-P 8850 7550
-F 0 "L7" H 8850 7855 60  0000 C CNN
-F 1 "TFM201208ALD-1R0MTCA" H 8850 7749 60  0000 C CNN
-F 2 "kria-k26-devboard-footprints:0603-res" H 9475 7900 60  0001 C CNN
-F 3 "https://product.tdk.com/system/files/dam/doc/product/inductor/inductor/smd/catalog/inductor_commercial_power_tfm201208ald_en.pdf" H 8905 7580 60  0001 C CNN
-F 4 "TDK" H 9000 8300 50  0001 C CNN "Manufacturer"
-F 5 "TFM201208ALD-1R0MTCA" H 9150 8200 50  0001 C CNN "MPN"
-F 6 "2.5A" H 8925 8100 50  0001 C CNN "MaxCur"
-F 7 "1.25x0.8" H 8975 8000 50  0001 C CNN "Size"
-F 8 "1u/2.5A" H 8850 7651 50  0000 C CNN "Val"
-	1    8850 7550
 	1    0    0    -1
 $EndComp
@@
 Wire Wire Line
 	4750 3450 4750 3400
+$Comp
+L antmicroFixedInductors:TFM201208ALD-1R0MTCA L4
+U 1 1 631602A4
+P 8850 2800
+F 0 "L4" H 8850 3105 60  0000 C CNN
+F 1 "TFM201208ALD-1R0MTCA" H 8850 2999 60  0000 C CNN
+F 2 "antmicro-footprints:0805-res" H 9475 3150 60  0001 C CNN
+F 3 "https://product.tdk.com/system/files/dam/doc/product/inductor/inductor/smd/catalog/inductor_commercial_power_tfm201208ald_en.pdf" H 8905 2830 60  0001 C CNN
+F 4 "TDK" H 9000 3550 50  0001 C CNN "Manufacturer"
+F 5 "TFM201208ALD-1R0MTCA" H 9150 3450 50  0001 C CNN "MPN"
+F 6 "2.5A" H 8925 3350 50  0001 C CNN "MaxCur"
+F 7 "1.25x0.8" H 8975 3250 50  0001 C CNN "Size"
+F 8 "1u/2.5A" H 8850 2901 50  0000 C CNN "Val"
+	1    8850 2800
+	1    0    0    -1
+$EndComp
+$Comp
+L antmicroFixedInductors:TFM201208ALD-1R0MTCA L7
+U 1 1 63193D9E
+P 8850 7550
+F 0 "L7" H 8850 7855 60  0000 C CNN
+F 1 "TFM201208ALD-1R0MTCA" H 8850 7749 60  0000 C CNN
+F 2 "antmicro-footprints:0805-res" H 9475 7900 60  0001 C CNN
+F 3 "https://product.tdk.com/system/files/dam/doc/product/inductor/inductor/smd/catalog/inductor_commercial_power_tfm201208ald_en.pdf" H 8905 7580 60  0001 C CNN
+F 4 "TDK" H 9000 8300 50  0001 C CNN "Manufacturer"
+F 5 "TFM201208ALD-1R0MTCA" H 9150 8200 50  0001 C CNN "MPN"
+F 6 "2.5A" H 8925 8100 50  0001 C CNN "MaxCur"
+F 7 "1.25x0.8" H 8975 8000 50  0001 C CNN "Size"
+F 8 "1u/2.5A" H 8850 7651 50  0000 C CNN "Val"
+	1    8850 7550
+	1    0    0    -1
+$EndComp
 $EndSCHEMATC
