File: eth.sch (KiCad schematic (older format))
At the start: 42 parts, among them J5 5-2337992-8, Q4 DTC014TEBTL, Q5 DTC014TEBTL, U30 DP83867CRRGZR, Y6 ECS-2016MV-250-CN-TR3

Commit message: Updated crystal library: fixed ECS-2016MV-240-BN-TR3 and ECS-2016MV-250-CN-TR3 MPN
Parts:
- Y6: footprint kria-k26-devboard-footprints:ECS-2016MV -> antmicro-footprints:ECS-2016MV; symbol kria-k26-devboard:ECS-2016MV-250-CN-TR3 -> antmicroCrystals:ECS-2016MV-250-CN-TR3; MPN ECS-2520MVLC-260-CM-TR -> ECS-2016MV-250-CN-TR3
Changed lines of the file:
@@
 	3200 8950 3200 8900
 $Comp
-L kria-k26-devboard:ECS-2016MV-250-CN-TR3 Y?
+L antmicroCrystals:ECS-2016MV-250-CN-TR3 Y?
 U 1 1 6317DA87
 P 4050 8700
@@
 F 0 "Y6" H 4250 8950 50  0000 L CNN
 F 1 "ECS-2016MV-250-CN-TR3" H 4100 8450 50  0000 L CNN
-F 2 "kria-k26-devboard-footprints:ECS-2016MV" H 4500 8350 50  0001 C CNN
+F 2 "antmicro-footprints:ECS-2016MV" H 4500 8350 50  0001 C CNN
 F 3 "https://www.mouser.pl/datasheet/2/122/ECS_2016MV-2529299.pdf" H 3875 8825 50  0001 C CNN
 F 4 "ECS" H 4200 8250 50  0001 C CNN "Manufacturer"
-F 5 "ECS-2520MVLC-260-CM-TR" H 4700 8150 50  0001 C CNN "MPN"
+F 5 "ECS-2016MV-250-CN-TR3" H 4700 8150 50  0001 C CNN "MPN"
 	1    4050 8700
 	1    0    0    -1
