File: usb.sch (KiCad schematic (older format))
At the start: 99 parts, among them U16 TPS2066TDGNRQ1, U17 USB7016_KDX, U18 TPS2066TDGNRQ1, U19 TPD4E05U06QDQARQ1_PASS, U20 WE-TVS-82400152, U21 WE-TVS-82400152, U22 TPD4E05U06QDQARQ1_PASS, U23 USB3310C-CP, U24 GSB3112311HR, U25 TPD4E05U06QDQARQ1_PASS, U26 WE-TVS-82400152, U27 WE-TVS-82400152, U28 TPD4E05U06QDQARQ1_PASS, U29 GSB3112311HR, Y4 ECS-2016MV-250-CN-TR3, Y5 ECS-2016MV-240-BN-TR3

Commit message: Updated crystal library: fixed ECS-2016MV-240-BN-TR3 and ECS-2016MV-250-CN-TR3 MPN
Parts:
- Y4: footprint kria-k26-devboard-footprints:ECS-2016MV -> antmicro-footprints:ECS-2016MV; symbol kria-k26-devboard:ECS-2016MV-250-CN-TR3 -> antmicroCrystals:ECS-2016MV-250-CN-TR3; MPN ECS-2520MVLC-260-CM-TR -> ECS-2016MV-250-CN-TR3
- Y5: footprint kria-k26-devboard-footprints:ECS-2016MV -> antmicro-footprints:ECS-2016MV; symbol kria-k26-devboard:ECS-2016MV-240-BN-TR3 -> antmicroCrystals:ECS-2016MV-240-BN-TR3; MPN ECS-2520MVLC-260-CM-TR -> ECS-2016MV-240-BN-TR3
Changed lines of the file:
@@
 USB power switches
 $Comp
-L kria-k26-devboard:ECS-2016MV-240-BN-TR3 Y5
+L antmicroCrystals:ECS-2016MV-240-BN-TR3 Y5
 U 1 1 63135142
 P 9800 3600
 F 0 "Y5" H 10000 3850 50  0000 L CNN
 F 1 "ECS-2016MV-240-BN-TR3" H 9950 3300 50  0000 L CNN
-F 2 "kria-k26-devboard-footprints:ECS-2016MV" H 10250 3250 50  0001 C CNN
+F 2 "antmicro-footprints:ECS-2016MV" H 10250 3250 50  0001 C CNN
 F 3 "https://www.mouser.pl/datasheet/2/122/ECS_2016MV-2529299.pdf" H 9625 3725 50  0001 C CNN
 F 4 "ECS" H 9950 3150 50  0001 C CNN "Manufacturer"
-F 5 "ECS-2520MVLC-260-CM-TR" H 10450 3050 50  0001 C CNN "MPN"
+F 5 "ECS-2016MV-240-BN-TR3" H 10450 3050 50  0001 C CNN "MPN"
 	1    9800 3600
 	1    0    0    -1
@@
 All ports removable
 $Comp
-L kria-k26-devboard:ECS-2016MV-250-CN-TR3 Y4
+L antmicroCrystals:ECS-2016MV-250-CN-TR3 Y4
 U 1 1 632C5A2B
 P 1400 4200
 F 0 "Y4" H 1600 4500 50  0000 L CNN
 F 1 "ECS-2016MV-250-CN-TR3" H 1500 3950 50  0000 L CNN
-F 2 "kria-k26-devboard-footprints:ECS-2016MV" H 1850 3850 50  0001 C CNN
+F 2 "antmicro-footprints:ECS-2016MV" H 1850 3850 50  0001 C CNN
 F 3 "https://www.mouser.pl/datasheet/2/122/ECS_2016MV-2529299.pdf" H 1225 4325 50  0001 C CNN
 F 4 "ECS" H 1550 3750 50  0001 C CNN "Manufacturer"
-F 5 "ECS-2520MVLC-260-CM-TR" H 2050 3650 50  0001 C CNN "MPN"
+F 5 "ECS-2016MV-250-CN-TR3" H 2050 3650 50  0001 C CNN "MPN"
 	1    1400 4200
 	1    0    0    -1
