File: kria-k26-devboard.kicad_sch (KiCad schematic)
At the start: 6 parts

Commit message: [#56935] Update symbol/footprint links; Migrate to KiCad 7
Parts:
- C1, C2: footprint kria-k26-devboard-footprints:C_0402_1005Metric -> antmicro-footprints:C_0402_1005Metric; symbol kria-k26-devboard:C_100n_0402 -> antmicroCapacitors0402:C_100n_0402
- N1: footprint kria-k26-devboard-footprints:antmicro-logo_scaled_30mm -> antmicro-footprints:antmicro-logo; symbol kria-k26-devboard:antmicro_logo -> antmicroMechanicalParts:antmicro_logo
- N2: footprint kria-k26-devboard-footprints:oshw-logo -> antmicro-footprints:oshw-logo; symbol kria-k26-devboard:oshw_logo -> antmicroMechanicalParts:oshw_logo
- R1, R2: footprint kria-k26-devboard-footprints:R_0402_1005Metric -> antmicro-footprints:R_0402_1005Metric; symbol kria-k26-devboard:R_330R_0402 -> antmicroResistors0402:R_330R_0402

Commit message: [#56935] Loclib
Parts:
- C1, C2: footprint antmicro-footprints:C_0402_1005Metric -> kria-k26-devboard-footprints:C_0402_1005Metric; symbol antmicroCapacitors0402:C_100n_0402 -> kria-k26-devboard:C_100n_0402
- N1: footprint antmicro-footprints:antmicro-logo -> kria-k26-devboard-footprints:antmicro-logo; symbol antmicroMechanicalParts:antmicro_logo -> kria-k26-devboard:antmicro_logo
- N2: footprint antmicro-footprints:oshw-logo -> kria-k26-devboard-footprints:oshw-logo; symbol antmicroMechanicalParts:oshw_logo -> kria-k26-devboard:oshw_logo
- R1, R2: footprint antmicro-footprints:R_0402_1005Metric -> kria-k26-devboard-footprints:R_0402_1005Metric; symbol antmicroResistors0402:R_330R_0402 -> kria-k26-devboard:R_330R_0402
Changed lines of the file:
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@@
     )
   )
-  (symbol (lib_id "antmicroResistors0402:R_330R_0402") (at 25.4 238.125 270) (unit 1)
+  (symbol (lib_id "kria-k26-devboard:R_330R_0402") (at 25.4 238.125 270) (unit 1)
     (in_bom yes) (on_board yes) (dnp no)
     (property "Reference" "R1" (at 26.67 239.3951 90)
@@
       (effects (font (size 1.27 1.27) (thickness 0.15)) (justify left bottom) hide)
     )
-    (property "Footprint" "antmicro-footprints:R_0402_1005Metric" (at 30.48 243.205 0)
+    (property "Footprint" "kria-k26-devboard-footprints:R_0402_1005Metric" (at 30.48 243.205 0)
       (effects (font (size 1.27 1.27) (thickness 0.15)) (justify left bottom) hide)
     )
@@
     )
   )
-  (symbol (lib_id "antmicroCapacitors0402:C_100n_0402") (at 33.02 238.125 270) (unit 1)
+  (symbol (lib_id "kria-k26-devboard:C_100n_0402") (at 33.02 238.125 270) (unit 1)
     (in_bom yes) (on_board yes) (dnp no)
     (property "Reference" "C1" (at 33.655 238.76 90)
@@
       (effects (font (size 1.27 1.27) (thickness 0.15)) (justify left bottom) hide)
     )
-    (property "Footprint" "antmicro-footprints:C_0402_1005Metric" (at 38.1 243.205 0)
+    (property "Footprint" "kria-k26-devboard-footprints:C_0402_1005Metric" (at 38.1 243.205 0)
       (effects (font (size 1.27 1.27) (thickness 0.15)) (justify left bottom) hide)
     )
@@
     )
   )
-  (symbol (lib_id "antmicropower:GND") (at 29.21 247.015 0) (unit 1)
+  (symbol (lib_id "kria-k26-devboard:GND") (at 29.21 247.015 0) (unit 1)
     (in_bom yes) (on_board yes) (dnp no)
     (property "Reference" "#PWR01" (at 29.21 253.365 0)
@@
     )
   )
-  (symbol (lib_id "antmicroResistors0402:R_330R_0402") (at 52.07 238.125 270) (unit 1)
+  (symbol (lib_id "kria-k26-devboard:R_330R_0402") (at 52.07 238.125 270) (unit 1)
     (in_bom yes) (on_board yes) (dnp no)
     (property "Reference" "R2" (at 53.34 239.3951 90)
@@
       (effects (font (size 1.27 1.27) (thickness 0.15)) (justify left bottom) hide)
     )
-    (property "Footprint" "antmicro-footprints:R_0402_1005Metric" (at 57.15 243.205 0)
+    (property "Footprint" "kria-k26-devboard-footprints:R_0402_1005Metric" (at 57.15 243.205 0)
       (effects (font (size 1.27 1.27) (thickness 0.15)) (justify left bottom) hide)
     )
@@
     )
   )
-  (symbol (lib_id "antmicroCapacitors0402:C_100n_0402") (at 59.69 238.125 270) (unit 1)
+  (symbol (lib_id "kria-k26-devboard:C_100n_0402") (at 59.69 238.125 270) (unit 1)
     (in_bom yes) (on_board yes) (dnp no)
     (property "Reference" "C2" (at 60.325 238.76 90)
@@
       (effects (font (size 1.27 1.27) (thickness 0.15)) (justify left bottom) hide)
     )
-    (property "Footprint" "antmicro-footprints:C_0402_1005Metric" (at 64.77 243.205 0)
+    (property "Footprint" "kria-k26-devboard-footprints:C_0402_1005Metric" (at 64.77 243.205 0)
       (effects (font (size 1.27 1.27) (thickness 0.15)) (justify left bottom) hide)
     )
@@
     )
   )
-  (symbol (lib_id "antmicropower:GND") (at 55.88 247.015 0) (unit 1)
+  (symbol (lib_id "kria-k26-devboard:GND") (at 55.88 247.015 0) (unit 1)
     (in_bom yes) (on_board yes) (dnp no)
     (property "Reference" "#PWR02" (at 55.88 253.365 0)
@@
     )
   )
-  (symbol (lib_id "antmicroMechanicalParts:oshw_logo") (at 52.07 262.89 0) (unit 1)
+  (symbol (lib_id "kria-k26-devboard:oshw_logo") (at 52.07 262.89 0) (unit 1)
     (in_bom yes) (on_board yes) (dnp no) (fields_autoplaced)
     (property "Reference" "N2" (at 58.42 260.5975 0)
@@
       (effects (font (size 1.27 1.27) (thickness 0.15)) (justify left))
     )
-    (property "Footprint" "antmicro-footprints:oshw-logo" (at 52.578 268.986 0)
+    (property "Footprint" "kria-k26-devboard-footprints:oshw-logo" (at 52.578 268.986 0)
       (effects (font (size 1.27 1.27) (thickness 0.15)) (justify left bottom) hide)
     )
@@
     )
   )
-  (symbol (lib_id "antmicroMechanicalParts:antmicro_logo") (at 25.4 262.89 0) (unit 1)
+  (symbol (lib_id "kria-k26-devboard:antmicro_logo") (at 25.4 262.89 0) (unit 1)
     (in_bom yes) (on_board yes) (dnp no) (fields_autoplaced)
     (property "Reference" "N1" (at 31.75 260.5975 0)
@@
       (effects (font (size 1.27 1.27) (thickness 0.15)) (justify left))
     )
-    (property "Footprint" "antmicro-footprints:antmicro-logo" (at 22.86 256.54 0)
-      (effects (font (size 1.27 1.27) (thickness 0.15)) (justify left bottom) hide)
-    )
+    (property "Footprint" "kria-k26-devboard-footprints:antmicro-logo" (at 22.86 256.54 0)
+      (effects (font (size 1.27 1.27) (thickness 0.15)) (justify left bottom) hide)
+    )
